File: schematic/sidpi.sch (EAGLE design)
At the start: 9 parts, among them IC1 7805T, J1 POWER_JACKPTH

Commit message: Updated schematic
Parts:
- removed J1: POWER_JACKPTH, SparkFun-Connectors:POWER_JACKPTH
- removed JP1: (no value), SparkFun-Connectors:AUDIO-JACKSPECIAL_POGO_PINS
- added CN1: 12V, adafruit:DCBARRELPTH
- added J2: AUDIO-JACK2KIT, SparkFun-Connectors:AUDIO-JACK2KIT
- C1: value (none) -> 2.2 NF
- C2: value (none) -> 2.2NF
Connections:
- removed net N$16: C3.-, JP1.LEFT, JP1.RIGHT
- new net N$8: C3.-, J2.RING, J2.TIP
- net GND: now also CN1.GND, CN1.GNDBREAK, J2.SLEEVE, SK1.GND@14, SK1.GND@20, SK1.GND@25, SK1.GND@9, U$1.R/W; no longer J1.PWR, U$1.RESET
- net VCC: now also U$1.RESET; no longer U$1.R/W
- net VDD: now also CN1.PWR; no longer J1.GND
Other:
- note added: "Version 1.0"
- moved on the sheet: C1, C2

Commit message: .
Other:
- note added: "Rev b"
Changed lines of the file:
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@@
 <frame x1="-294.64" y1="124.46" x2="-12.7" y2="266.7" columns="8" rows="5" layer="91"/>
 <text x="-233.68" y="162.56" size="1.778" layer="91">Version 1.0</text>
+<text x="-228.6" y="157.48" size="1.778" layer="91">Rev b</text>
 </plain>
 <instances>
